Commit message: feat: Hibrid NLP (Ses/Yazı) otonom kontrolü, MediaPipe AI entegrasyonu ve 6 eksenli (6-DOF) cobot çarpışma fiziği eklendi 🚀

File: src/rokisim_gazebo/urdf/simple_arm.urdf (robot description, URDF)
Before this commit: robot rokisim_6dof_cobot, 11 links, 10 joints
Links:
- removed link gripper_jaw
- added link finger_left, mass 0.05; collision box size=0.015 0.03 0.10; visual box size=0.015 0.03 0.10
- added link finger_right, mass 0.05; collision box size=0.015 0.03 0.10; visual box size=0.015 0.03 0.10
- added link gripper_base, mass 0.2; collision box size=0.16 0.04 0.04; visual box size=0.16 0.04 0.04
- link link1: geometry collision cylinder length=0.2 radius=0.07; visual cylinder length=0.2 radius=0.07
- link link2: geometry collision cylinder length=0.4 radius=0.06; visual cylinder length=0.4 radius=0.06
- link link3: geometry collision cylinder length=0.3 radius=0.05; visual cylinder length=0.3 radius=0.05
- link link4: geometry collision cylinder length=0.1 radius=0.04; visual cylinder length=0.1 radius=0.04
- link link5: geometry collision cylinder length=0.1 radius=0.035; visual cylinder length=0.1 radius=0.035
- link link6: geometry collision cylinder length=0.05 radius=0.03; visual cylinder length=0.05 radius=0.03
Joints:
- added joint gripper_base_joint: type fixed, parent link6, child gripper_base, origin xyz=0 0 0.05 rpy=0 0 0
- added joint gripper_right_joint: type fixed, parent gripper_base, child finger_right, origin xyz=-0.07 0 0.04 rpy=0 0 0
- joint gripper_joint: axis 1 0 0 -> -1 0 0; child gripper_jaw -> finger_left; limit lower=0.0 upper=0.05 effort=20 velocity=0.5 -> lower=0.0 upper=0.125 effort=100 velocity=0.5; origin xyz=0 0 0.05 rpy=0 0 0 -> xyz=0.07 0 0.04 rpy=0 0 0; parent link6 -> gripper_base

Commit message: feat: J.A.R.V.I.S. tabanlı İngilizce erkek TTS (Text-to-Speech) durum bildirim motoru eklendi 🎙️

File: src/rokisim_gazebo/urdf/simple_arm.urdf (robot description, URDF)
Before this commit: robot rokisim_6dof_cobot, 13 links, 12 joints
Joints:
- joint joint1: limit lower=-3.14 upper=3.14 effort=150 velocity=3.15 -> lower=-2.8 upper=2.8 effort=150 velocity=1.5
- joint joint2: limit lower=-3.14 upper=3.14 effort=150 velocity=3.15 -> lower=-1.57 upper=1.57 effort=150 velocity=1.5
- joint joint3: limit lower=-3.14 upper=3.14 effort=150 velocity=3.15 -> lower=-2.45 upper=2.45 effort=150 velocity=2.0
- joint joint4: limit lower=-3.14 upper=3.14 effort=50 velocity=3.15 -> lower=-1.57 upper=1.57 effort=50 velocity=2.5
